Commit message: obstacle detection and fixed distance test

File: src/rover_pkg/urdf/rover.urdf.xacro (robot description, xacro)
@@ -5,4 +5,9 @@
     <!-- <link name="${proper}"/> -->
     <!-- Materials -->
+    <xacro:arg name="odom_frame" default="odom"/>
+    <xacro:arg name="base_footprint" default="base_footprint"/>
+    <xacro:arg name="base_stabilized" default="base_stabilized"/>
+    <xacro:arg name="base_frame" default="base_link"/>
+    <xacro:arg name="lase_frame" default="laser"/>
     <material name="black">
         <color rgba="0 0 0 1"/>
@@ -18,7 +23,18 @@
     </material>
     <!-- Map link -->
-    <link name="map" >
+    <link name="map" />
+    <!-- Base foot print -->
+    <link name="$(arg base_footprint)" />
+    <joint name="$(arg base_footprint)_to_map_joint" type="fixed">
         <origin xyz="0.0 0.0 0.0" rpy="0.0 0.0 0.0"/>
-    </link>
+        <parent link="map"/>
+        <child link="$(arg base_footprint)"/>
+    </joint>
+    <link name="$(arg base_stabilized)" />
+    <joint name="$(arg base_stabilized)_to_$(arg base_footprint)_joint" type="fixed">
+        <origin xyz="0.0 0.0 0.14" rpy="0.0 0.0 0.0"/>
+        <parent link="$(arg base_footprint)"/>
+        <child link="$(arg base_stabilized)"/>
+    </joint>
     <!-- List of 3D inertia tensors: https://en.wikipedia.org/wiki/List_of_moments_of_inertia#List_of_3D_inertia_tensors -->
     <!-- To calculate inertia on baselink-->
@@ -32,5 +48,5 @@
     <xacro:property name="scale" value="0.001"/> <!-- This works for base_link and laser links, helps to scale them propertly-->
     <!-- Base link -->
-    <link name="base_link">
+    <link name="$(arg base_frame)">
         <inertial>  <!--Inertial model for simulation on GAZEBO -->
             <origin xyz="-0.004 0.0 0.009" rpy="0.0 0.0 0.0"/>
@@ -57,9 +73,8 @@
         </collision>
     </link>
-    <joint name="base_joint" type="fixed">
-        <origin xyz="0.0 0.0 0.14" rpy="0.0 0.0 0.0"/>
-        <parent link="map"/>
-        <child link="base_link"/>
-        <axis xyz="0.0 0.0 0.0"/>
+    <joint name="$(arg base_frame)_joint" type="fixed">
+        <origin xyz="0.0 0.0 0.0" rpy="0.0 0.0 0.0"/>
+        <parent link="$(arg base_stabilized)"/>
+        <child link="$(arg base_frame)"/>
     </joint>
     <xacro:macro name="wheel" params="name x y z">
@@ -89,5 +104,5 @@
         <joint name="${name}_wheel_joint" type="fixed">
             <origin xyz="${x} ${y} ${z}" rpy="0.0 0.0 0.0"/>
-            <parent link="base_link"/>
+            <parent link="$(arg base_frame)"/>
             <child link="${name}_wheel_link"/>
             <!-- <axis xyz="0.0 1.0 0.0"/> -->
@@ -116,5 +131,5 @@
     <xacro:property name="laser_depth" value="0.07"/>
     <!-- Laser link -->
-    <link name="laser">
+    <link name="$(arg lase_frame)">
         <inertial>
             <origin xyz="0.0 0.0 0.0" rpy="0.0 0.0 0.0"/>
@@ -126,5 +141,5 @@
         <visual>
             <!-- <origin xyz="1.2 1.7 0.5" rpy="0.0 0.0 0.0"/> -->
-            <origin xyz="0.035 -0.035 -0.035" rpy="${pi/2.0} 0.0 ${pi}"/>
+            <origin xyz="-0.035 0.035 -0.035" rpy="${pi/2} 0.0 0.0"/>
             <geometry>
                 <mesh filename="package://rover_pkg/meshes/rplidar_main.stl" scale="${scale} ${scale} ${scale}"/>
@@ -141,9 +156,9 @@
         </collision>
     </link>
-    <joint name="laser_joint" type="fixed">
+    <joint name="$(arg lase_frame)_joint" type="fixed">
         <!-- <origin xyz="0.0 0.0 0.13" rpy="0.0 0.0 0.0"/> -->
-        <origin xyz="0.0 0.0 0.15" rpy="0.0 0.0 0.0"/>
-        <parent link="base_link"/>
-        <child link="laser"/>
+        <origin xyz="0.0 0.0 0.15" rpy="0.0 0.0 ${pi}"/>
+        <parent link="$(arg base_frame)"/>
+        <child link="$(arg lase_frame)"/>
         <axis xyz="0.0 0.0 0.0"/>
     </joint>
